File: H1_Jetson_AGX_Orin_SOM/EthernetIf.kicad_sch (KiCad schematic)
At the start: 36 parts, among them J4 SIM_Card_Shielded, J5 RJ45_JK0654219, U4 RG520N, U6 KSZ9031RNXCA, Y3 25Mhz Crystal

Commit message: Integrated all schematics and PCB files into a single directory for H1_Jetson_AGX_Orin_SOM project.
Parts:
- renumbered 0R to 0R1, 0R to 0R2, 0R to 0R3, AE3 to AE2, AE2 to AE3, C13 to C56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
Other:
- company: (none) -> Bosch Global Software Techonlogies
- title: (none) -> Humanoid-H1
