File: H1_Jetson_AGX_Orin_SOM/WifiIf.kicad_sch (KiCad schematic)
At the start: 47 parts, among them J1 Bus_M.2_1-2199230-6, J2 4-pin Molex 53261-0471, J3 Bus_M.2_2199230-6, Q1 Q_NMOS_GDS, Y2 Oscillator_32.768kHz_ECS_2520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

Commit message: Integrated all schematics and PCB files into a single directory for H1_Jetson_AGX_Orin_SOM project.
Parts:
- gave numbers to parts that had none: 3
- renumbered C30 to C68, C31 to C69, C32 to C70, C25 to C71, C5 to C72, C7 to C73, C11 to C74, C9 to C75, C6 to C76, C8 to C77, C12 to C78, C10 to C79, C21 to C80, C1 to C81, C2 to C82, C22 to C83, C23 to C84, C24 to C85, C3 to C86, C4 to C87, D3 to D13, D1 to D14, D2 to D15, J3 to J10, J2 to J8, J1 to J9, Q1 to Q10, R143 to R100, R2 to R101, R3 to R102, R4 to R103, R13 to R90, R14 to R91, R5 to R92, R15 to R93, R16 to R94, R12 to R95, R17 to R96, R1 to R98, R39 to R99, U1 to U20, U3 to U22, U2 to U23
Other:
- note added: "PCIe0 1x4 key M NVMe SSD"
- note added: "PCIe1 1x1 key E Wifi"
- note removed: "PCIe0 1x4 key M"
- company: (none) -> Bosch Global Software Techonlogies
- title: (none) -> Humanoid-H1
- moved on the sheet: C68, C69, C70, C71, C72, C73, C74, C75, C76, C77, C78, C79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
